File: mainboard.sch (KiCad schematic (older format))
At the start: 135 parts, among them J1 PAD, J10 PAD, J11 Conn_02x05_Odd_Even_MountingP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, J12 Conn_02x05_Odd_Even_MountingP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, J13 PAD, J14 PAD, J15 PAD, J16 PAD, J2 PAD, J3 PAD, J4 PAD, J5 PAD, J6 PAD, J7 PAD, J8 PAD, J9 PAD, Q1 CSD75208W1015, Q2 CSD75208W1015, Q3 CSD75208W1015, Q4 2N7002, U1 SX1261, U10 TPS61099, U11 TMUX1209, U12 TMUX1209, U13 OPA333xxDCK, U2 PE4259, U3 REF3020, U4 STM32L072CBYx, U5 TMUX1209, U6 LPV542, U7 LMT70, U8 TMUX1209, U9 LPV542, Y1 32MHz

Commit message: finished routing
Parts:
- added C51: 100n, Capacitor_SMD:C_0201_0603Metric, symbol Device:C_Small
Connections:
- net GNDA is gone; now on net GNDD: C13.2, C21.1, C29.1, R21.2, R6.2, U3.3 (GND), U7.A1 (GND)
- net RF_CLK is gone; now on net RF_SCK: U4.A3 (PB3)
- net +5VA: now also C42.1, C43.1, C51.1
- net ADC_IN12: now also R33.2; no longer R38.2
- net ADC_IN3: now also R27.2; no longer R19.2
- net ADC_IN6: now also R19.2; no longer R37.2
- net ADC_IN7: now also R37.2; no longer R27.2
- net ADC_IN9: now also R38.2; no longer R33.2
- net AFE_EN: now also U4.E1 (PB15)
- net ANT_SW: now also U4.B7 (PC13)
- net DAC_OUT1: now also R12.2, R28.2; no longer U13.1 (+)
- net DAC_OUT2: now also U13.1 (+); no longer R12.2, R28.2
- net GNDD: now also C51.2
- net ISFET2_D1: now also J4.1 (Pin_1); no longer J10.1 (Pin_1)
- net ISFET2_D2: now also J1.1 (Pin_1); no longer J9.1 (Pin_1)
- net ISFET2_D3: now also J2.1 (Pin_1); no longer J7.1 (Pin_1)
- net ISFET2_D4: now also J3.1 (Pin_1); no longer J5.1 (Pin_1)
- net MUX1IN0: now also U4.F2 (PB13), U8.15 (A0); no longer U5.15 (A0)
- net MUX1IN1: now also U4.G1 (PB12), U8.14 (A1); no longer U5.14 (A1)
- net MUX2IN0: now also U5.15 (A0); no longer U8.15 (A0)
- net MUX2IN1: now also U5.14 (A1); no longer U8.14 (A1)
- net MUX3EN: now also U4.E2 (PA9)
- net MUX3IN0: now also U4.F3 (PB11)
- net MUX3IN1: now also U4.C1 (PA10)
- net MUX4IN0: now also U4.A6 (PB9)
- net MUX4IN1: now also U4.B5 (PB8)
- net REFFET1_D1: now also J12.10 (Pin_10); no longer J12.4 (Pin_4)
- net REFFET1_D2: now also J12.8 (Pin_8); no longer J12.6 (Pin_6)
- net REFFET1_D3: now also J12.6 (Pin_6); no longer J12.8 (Pin_8)
- net REFFET1_D4: now also J12.4 (Pin_4); no longer J12.10 (Pin_10)
- net REFFET2_D1: now also J5.1 (Pin_1); no longer J1.1 (Pin_1)
- net REFFET2_D2: now also J7.1 (Pin_1); no longer J2.1 (Pin_1)
- net REFFET2_D3: now also J9.1 (Pin_1); no longer J3.1 (Pin_1)
- net REFFET2_D4: now also J10.1 (Pin_1); no longer J4.1 (Pin_1)
- net RF_BUSY: now also U4.D2 (PA11)
- net RF_RST: now also U4.D1 (PA8)
- net TAG_EN: now also U4.F1 (PB14)
- net VCC: no longer C42.1, C43.1
Other:
- moved on the sheet: C42, C43, R19, R27, R33, R37, R38
